File: Grove-Base-for-ESPr-Developer.sch (EAGLE design)
At the start: 8 parts, among them J1 4P-2.0, J2 4P-2.0, J3 4P-2.0, J4 4P-2.0

Commit message: 1st 5V evt
Parts:
- added R10, R11, R12, R13, R14, R3, R4, R5, R6, R7, R8, R9: 1K, Seeed-OPL-Resistor:SMD-RES-220K-1%-1/10W(0603)
- added R15: 27K, Seeed-OPL-Resistor:SMD-RES-100K-1%-1/10W(0603)
- added T1, T2, T3, T4, T5, T6: (no value), we-transistor:MOSFET-N-SOT23
- R1: value 220K -> 200K
- R2: value 100K -> 24K
Connections:
- new net IO12_5V: J2.1, R8.1, T3.D
- new net IO13_5V: J2.2, R10.2, T4.D
- new net IO14_5V: J1.1, R4.2, T1.D
- new net IO15_5V: J1.2, R6.2, T2.D
- new net IO4_5V: J4.2, R14.2, T6.D
- new net IO5_5V: J4.1, R12.1, T5.D
- new net N$6: R15.2, R2.1
- net 3V3: now also R11.2, R13.1, R3.1, R5.1, R7.2, R9.1, T1.G, T2.G, T3.G, T4.G, T5.G, T6.G; no longer J1.3, J2.3, J3.3, J4.3
- net 5V: now also J1.3, J2.3, J3.3, J4.3, R10.1, R12.2, R14.1, R4.1, R6.1, R8.2
- net GND: now also R15.1; no longer R2.1
- net IO12: now also R7.1, T3.S; no longer J2.1
- net IO13: now also R9.2, T4.S; no longer J2.2
- net IO14: now also R3.2, T1.S; no longer J1.1
- net IO15: now also R5.2, T2.S; no longer J1.2
- net IO4: now also R13.2, T6.S; no longer J4.2
- net IO5: now also R11.1, T5.S; no longer J4.1
Other:
- moved on the sheet: J1, J2, J3, J4, JP1, JP2, R1, R2

Commit message: 2nd EVT
2nd EVT (for hand soldering...)
Parts:
- removed R3, R4, R5, R6: 1K, Seeed-OPL-Resistor:SMD-RES-220K-1%-1/10W(0603)
- removed T1, T2: (no value), we-transistor:MOSFET-N-SOT23
- R10, R11, R12, R13, R14, R7, R8, R9: value 1K -> 10K
Connections:
- removed net IO14_5V: J1.1, R4.2, T1.D
- removed net IO15_5V: J1.2, R6.2, T2.D
- net 3V3: now also J1.3; no longer R3.1, R5.1, T1.G, T2.G
- net 5V: no longer J1.3, R4.1, R6.1
- net IO14: now also J1.1; no longer R3.2, T1.S
- net IO15: now also J1.2; no longer R5.2, T2.S
Changed lines of the file:
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@@
 <part name="GND" library="supply1" deviceset="GND" device=""/>
 <part name="FRAME1" library="frames" deviceset="DINA5_L" device=""/>
-<part name="T1" library="we-transistor" deviceset="MOSFET-N" device="-SOT23"/>
-<part name="T2" library="we-transistor" deviceset="MOSFET-N" device="-SOT23"/>
 <part name="T3" library="we-transistor" deviceset="MOSFET-N" device="-SOT23"/>
 <part name="T4" library="we-transistor" deviceset="MOSFET-N" device="-SOT23"/>
@@
 <part name="T6" library="we-transistor" deviceset="MOSFET-N" device="-SOT23"/>
 <part name="R15" library="Seeed-OPL-Resistor" deviceset="SMD-RES-100K-1%-1/10W(0603)" device="" value="27K"/>
-<part name="R3" library="Seeed-OPL-Resistor" deviceset="SMD-RES-220K-1%-1/10W(0603)" device="" value="1K"/>
-<part name="R4" library="Seeed-OPL-Resistor" deviceset="SMD-RES-220K-1%-1/10W(0603)" device="" value="1K"/>
-<part name="R5" library="Seeed-OPL-Resistor" deviceset="SMD-RES-220K-1%-1/10W(0603)" device="" value="1K"/>
-<part name="R6" library="Seeed-OPL-Resistor" deviceset="SMD-RES-220K-1%-1/10W(0603)" device="" value="1K"/>
-<part name="R7" library="Seeed-OPL-Resistor" deviceset="SMD-RES-220K-1%-1/10W(0603)" device="" value="1K"/>
-<part name="R8" library="Seeed-OPL-Resistor" deviceset="SMD-RES-220K-1%-1/10W(0603)" device="" value="1K"/>
-<part name="R9" library="Seeed-OPL-Resistor" deviceset="SMD-RES-220K-1%-1/10W(0603)" device="" value="1K"/>
-<part name="R10" library="Seeed-OPL-Resistor" deviceset="SMD-RES-220K-1%-1/10W(0603)" device="" value="1K"/>
-<part name="R11" library="Seeed-OPL-Resistor" deviceset="SMD-RES-220K-1%-1/10W(0603)" device="" value="1K"/>
-<part name="R12" library="Seeed-OPL-Resistor" deviceset="SMD-RES-220K-1%-1/10W(0603)" device="" value="1K"/>
-<part name="R13" library="Seeed-OPL-Resistor" deviceset="SMD-RES-220K-1%-1/10W(0603)" device="" value="1K"/>
-<part name="R14" library="Seeed-OPL-Resistor" deviceset="SMD-RES-220K-1%-1/10W(0603)" device="" value="1K"/>
+<part name="R7" library="Seeed-OPL-Resistor" deviceset="SMD-RES-220K-1%-1/10W(0603)" device="" value="10K"/>
+<part name="R8" library="Seeed-OPL-Resistor" deviceset="SMD-RES-220K-1%-1/10W(0603)" device="" value="10K"/>
+<part name="R9" library="Seeed-OPL-Resistor" deviceset="SMD-RES-220K-1%-1/10W(0603)" device="" value="10K"/>
+<part name="R10" library="Seeed-OPL-Resistor" deviceset="SMD-RES-220K-1%-1/10W(0603)" device="" value="10K"/>
+<part name="R11" library="Seeed-OPL-Resistor" deviceset="SMD-RES-220K-1%-1/10W(0603)" device="" value="10K"/>
+<part name="R12" library="Seeed-OPL-Resistor" deviceset="SMD-RES-220K-1%-1/10W(0603)" device="" value="10K"/>
+<part name="R13" library="Seeed-OPL-Resistor" deviceset="SMD-RES-220K-1%-1/10W(0603)" device="" value="10K"/>
+<part name="R14" library="Seeed-OPL-Resistor" deviceset="SMD-RES-220K-1%-1/10W(0603)" device="" value="10K"/>
 </parts>
 <sheets>
@@
 <instance part="GND" gate="1" x="50.8" y="60.96"/>
 <instance part="FRAME1" gate="G$1" x="0" y="0"/>
-<instance part="T1" gate="T" x="101.6" y="78.74"/>
-<instance part="T2" gate="T" x="101.6" y="45.72"/>
 <instance part="T3" gate="T" x="129.54" y="78.74"/>
 <instance part="T4" gate="T" x="129.54" y="45.72"/>
@@
 <instance part="T6" gate="T" x="157.48" y="45.72"/>
 <instance part="R15" gate="G$1" x="50.8" y="71.12" rot="R90"/>
-<instance part="R3" gate="G$1" x="101.6" y="66.04" rot="R90"/>
-<instance part="R4" gate="G$1" x="109.22" y="86.36" rot="R180"/>
-<instance part="R5" gate="G$1" x="101.6" y="33.02" rot="R90"/>
-<instance part="R6" gate="G$1" x="109.22" y="53.34" rot="R180"/>
 <instance part="R7" gate="G$1" x="129.54" y="66.04" rot="R270"/>
 <instance part="R8" gate="G$1" x="137.16" y="86.36"/>
@@
 </segment>
 <segment>
-<pinref part="T2" gate="T" pin="S"/>
-<wire x1="101.6" y1="36.83" x2="101.6" y2="38.1" width="0.1524" layer="91"/>
-<pinref part="R5" gate="G$1" pin="2"/>
-<wire x1="101.6" y1="38.1" x2="101.6" y2="40.64" width="0.1524" layer="91"/>
-<wire x1="101.6" y1="38.1" x2="109.22" y2="38.1" width="0.1524" layer="91"/>
-<junction x="101.6" y="38.1"/>
-<label x="104.14" y="38.1" size="1.778" layer="95"/>
-<label x="104.14" y="38.1" size="1.778" layer="95"/>
+<pinref part="J1" gate="G$1" pin="2"/>
+<wire x1="8.89" y1="106.68" x2="19.05" y2="106.68" width="0.1524" layer="91"/>
+<label x="8.89" y="106.68" size="1.778" layer="95"/>
 </segment>
 </net>
@@
 </segment>
 <segment>
-<pinref part="T1" gate="T" pin="S"/>
-<wire x1="101.6" y1="69.85" x2="101.6" y2="71.12" width="0.1524" layer="91"/>
-<pinref part="R3" gate="G$1" pin="2"/>
-<wire x1="101.6" y1="71.12" x2="101.6" y2="73.66" width="0.1524" layer="91"/>
-<wire x1="101.6" y1="71.12" x2="109.22" y2="71.12" width="0.1524" layer="91"/>
-<junction x="101.6" y="71.12"/>
-<label x="104.14" y="71.12" size="1.778" layer="95"/>
+<pinref part="J1" gate="G$1" pin="1"/>
+<wire x1="8.89" y1="109.22" x2="19.05" y2="109.22" width="0.1524" layer="91"/>
+<label x="8.89" y="109.22" size="1.778" layer="95"/>
 </segment>
 </net>
@@
 </segment>
 <segment>
-<wire x1="119.38" y1="53.34" x2="113.03" y2="53.34" width="0.1524" layer="91"/>
-<label x="119.38" y="55.88" size="1.778" layer="95" rot="R180"/>
-<pinref part="R6" gate="G$1" pin="1"/>
-</segment>
-<segment>
 <wire x1="149.86" y1="53.34" x2="140.97" y2="53.34" width="0.1524" layer="91"/>
 <label x="149.86" y="55.88" size="1.778" layer="95" rot="R180"/>
@@
 </segment>
 <segment>
-<wire x1="119.38" y1="86.36" x2="113.03" y2="86.36" width="0.1524" layer="91"/>
-<label x="119.38" y="88.9" size="1.778" layer="95" rot="R180"/>
-<label x="119.38" y="88.9" size="1.778" layer="95" rot="R180"/>
-<pinref part="R4" gate="G$1" pin="1"/>
-</segment>
-<segment>
 <wire x1="140.97" y1="86.36" x2="149.86" y2="86.36" width="0.1524" layer="91"/>
 <label x="149.86" y="88.9" size="1.778" layer="95" rot="R180"/>
 <pinref part="R8" gate="G$1" pin="2"/>
-</segment>
-<segment>
-<pinref part="J1" gate="G$1" pin="3"/>
-<wire x1="8.89" y1="104.14" x2="19.05" y2="104.14" width="0.1524" layer="91"/>
-<label x="8.89" y="104.14" size="1.778" layer="95"/>
 </segment>
 <segment>
@@
 <wire x1="11.43" y1="21.59" x2="19.05" y2="21.59" width="0.1524" layer="91"/>
 <label x="11.43" y="21.59" size="1.778" layer="95"/>
-</segment>
-<segment>
-<pinref part="T1" gate="T" pin="G"/>
-<wire x1="96.52" y1="76.2" x2="93.98" y2="76.2" width="0.1524" layer="91"/>
-<label x="88.9" y="76.2" size="1.778" layer="95"/>
-<wire x1="93.98" y1="76.2" x2="88.9" y2="76.2" width="0.1524" layer="91"/>
-<wire x1="93.98" y1="76.2" x2="93.98" y2="60.96" width="0.1524" layer="91"/>
-<wire x1="93.98" y1="60.96" x2="101.6" y2="60.96" width="0.1524" layer="91"/>
-<junction x="93.98" y="76.2"/>
-<wire x1="101.6" y1="60.96" x2="101.6" y2="62.23" width="0.1524" layer="91"/>
-<pinref part="R3" gate="G$1" pin="1"/>
-</segment>
-<segment>
-<pinref part="T2" gate="T" pin="G"/>
-<wire x1="96.52" y1="43.18" x2="93.98" y2="43.18" width="0.1524" layer="91"/>
-<label x="88.9" y="43.18" size="1.778" layer="95"/>
-<wire x1="93.98" y1="43.18" x2="88.9" y2="43.18" width="0.1524" layer="91"/>
-<wire x1="93.98" y1="43.18" x2="93.98" y2="27.94" width="0.1524" layer="91"/>
-<wire x1="93.98" y1="27.94" x2="101.6" y2="27.94" width="0.1524" layer="91"/>
-<junction x="93.98" y="43.18"/>
-<wire x1="101.6" y1="29.21" x2="101.6" y2="27.94" width="0.1524" layer="91"/>
-<pinref part="R5" gate="G$1" pin="1"/>
 </segment>
 <segment>
@@
 <pinref part="R13" gate="G$1" pin="1"/>
 </segment>
+<segment>
+<pinref part="J1" gate="G$1" pin="3"/>
+<wire x1="8.89" y1="104.14" x2="19.05" y2="104.14" width="0.1524" layer="91"/>
+<label x="8.89" y="104.14" size="1.778" layer="95"/>
+</segment>
 </net>
 <net name="N$6" class="0">
@@
 </segment>
 </net>
-<net name="IO14_5V" class="0">
-<segment>
-<pinref part="J1" gate="G$1" pin="1"/>
-<wire x1="8.89" y1="109.22" x2="19.05" y2="109.22" width="0.1524" layer="91"/>
-<label x="8.89" y="109.22" size="1.778" layer="95"/>
-</segment>
-<segment>
-<wire x1="105.41" y1="86.36" x2="101.6" y2="86.36" width="0.1524" layer="91"/>
-<wire x1="101.6" y1="86.36" x2="101.6" y2="88.9" width="0.1524" layer="91"/>
-<wire x1="101.6" y1="88.9" x2="109.22" y2="88.9" width="0.1524" layer="91"/>
-<pinref part="T1" gate="T" pin="D"/>
-<wire x1="101.6" y1="83.82" x2="101.6" y2="86.36" width="0.1524" layer="91"/>
-<junction x="101.6" y="86.36"/>
-<label x="109.22" y="91.44" size="1.778" layer="95" rot="R180"/>
-<pinref part="R4" gate="G$1" pin="2"/>
-</segment>
-</net>
-<net name="IO15_5V" class="0">
-<segment>
-<pinref part="J1" gate="G$1" pin="2"/>
-<wire x1="8.89" y1="106.68" x2="19.05" y2="106.68" width="0.1524" layer="91"/>
-<label x="8.89" y="106.68" size="1.778" layer="95"/>
-</segment>
-<segment>
-<wire x1="105.41" y1="53.34" x2="101.6" y2="53.34" width="0.1524" layer="91"/>
-<pinref part="T2" gate="T" pin="D"/>
-<wire x1="101.6" y1="53.34" x2="101.6" y2="50.8" width="0.1524" layer="91"/>
-<wire x1="101.6" y1="53.34" x2="101.6" y2="55.88" width="0.1524" layer="91"/>
-<wire x1="101.6" y1="55.88" x2="109.22" y2="55.88" width="0.1524" layer="91"/>
-<junction x="101.6" y="53.34"/>
-<label x="109.22" y="58.42" size="1.778" layer="95" rot="R180"/>
-<pinref part="R6" gate="G$1" pin="2"/>
-</segment>
-</net>
